File: sch/foxcar-control-board-v1.sch (EAGLE design)
At the start: 114 parts, among them J1 USB_MICROB_PLUG-PTH, J2 MICROSD, J3 XBEE-PRO, U1 SPX29300, U2 HMC5883LSMD, U3 STM32F4V, U4 VNH5019, U6 MPU6000

Commit message: Layout done, screenshots uploaded, parts list added.
Parts:
- removed JP21, JP22, JP23, JP24: M01PTH, SparkFun-Connectors:M01PTH
- removed JP25, JP26, JP27, JP28, JP29, JP30, JP31, JP32, JP33, JP34, JP35, JP36, JP37, JP38, JP39, JP40, JP41, JP42, JP43: M01PTH_LONGPAD, SparkFun-Connectors:M01PTH_LONGPAD
- removed R20: 4.7k, SparkFun-Passives:RESISTOR0402-RES
- removed TP10, TP11, TP13, TP3, TP4, TP8, TP9: TPTP06R, testpad:TPTP06R
- removed U6: MPU6000, invensense:MPU-6000
- added R9: 1k, SparkFun-Passives:RESISTOR0402-RES
- added U5: STM32F4V, stm32f4:STM32F4V_100PIN_FOXCAR
- C10: value 100nF -> 2.2uF
- C11: value 100nF -> 4.7uF; device SparkFun-Passives:CAP0402-CAP -> SparkFun-Passives:CAP0805
- C12: value 0.1uF -> 0.22uF
- C13: value 33nF -> 0.22uF
- C14, C15: value 0.22uF -> 2.2uF; device SparkFun-Passives:CAP0402-CAP -> SparkFun-Passives:CAP0603-CAP
- C16: value 4.7uF -> 16pF; device SparkFun-Passives:CAP0805 -> SparkFun-Passives:CAP0402-CAP
- C17, C22: value 0.1uF -> 100nF
- C18, C23: value 2.2uF -> 100nF; device SparkFun-Passives:CAP0603-CAP -> SparkFun-Passives:CAP0402-CAP
- C19: value 2.2uF -> 16pF
- C2: value 0.1uF -> 33nF
- C24: value 10nF -> 100nF
- C3: value 47uF -> 0.1uF; device SparkFun-Passives:CAP0805 -> SparkFun-Passives:CAP0402-CAP
- C4: value 16pF -> 10u; device SparkFun-Passives:CAP0402-CAP -> SparkFun-Passives:CAP0603-CAP
- C5: value 16pF -> 47uF; device SparkFun-Passives:CAP0402-CAP -> SparkFun-Passives:CAP0805
- C6: value 10u -> 0.1uF; device SparkFun-Passives:CAP0603-CAP -> SparkFun-Passives:CAP0402-CAP
- C7, C8: value 100nF -> 0.1uF
- C9: value 100nF -> 10nF
- J1: value USB_MICROB_PLUG-PTH -> MICROSD; device SparkFun:USB_MICROB_PLUG-PTH -> adafruit:MICROSD
- J2: value MICROSD -> XBEE-PRO; device adafruit:MICROSD -> maxstream:XBEE-PRO
- J3: value XBEE-PRO -> USB_MICROB_PLUG-PTH; device maxstream:XBEE-PRO -> SparkFun:USB_MICROB_PLUG-PTH
- JP1: value M01PTH_LONGPAD -> BATT; device SparkFun-Connectors:M01PTH_LONGPAD -> SparkFun-Connectors:M023.5MM_LOCK
- JP10: value M01PTH_LONGPAD -> UART2; device SparkFun-Connectors:M01PTH_LONGPAD -> SparkFun-Connectors:M04LOCK_LONGPADS
- JP11: value ESCD -> I2C1-B; device SparkFun-Connectors:M03LOCK_LONGPADS -> SparkFun-Connectors:M04LOCK_LONGPADS
- JP12: value ESCC -> USART3; device SparkFun-Connectors:M03LOCK_LONGPADS -> SparkFun-Connectors:M04LOCK_LONGPADS
- JP13: value ESCB -> SPI1; device SparkFun-Connectors:M03LOCK_LONGPADS -> SparkFun-Connectors:M06LOCK_LONGPADS
- JP14: value ESCA -> (none); device SparkFun-Connectors:M03LOCK_LONGPADS -> SparkFun-Connectors:M04LOCK
- JP15: value USART3 -> M01PTH; device SparkFun-Connectors:M04LOCK_LONGPADS -> SparkFun-Connectors:M01PTH
- JP16: value M01PTH -> (none); device SparkFun-Connectors:M01PTH -> SparkFun-Connectors:M02LOCK_LONGPADS
- JP17: value M01PTH -> (none); device SparkFun-Connectors:M01PTH -> SparkFun-Connectors:M07LOCK
- JP18: value M01PTH -> (none); device SparkFun-Connectors:M01PTH -> SparkFun-Connectors:M08LOCK_LONGPADS
- JP19: value M01PTH -> (none); device SparkFun-Connectors:M01PTH -> SparkFun-Connectors:M02LOCK
- JP2: value USART1 -> MOTORS; device SparkFun-Connectors:M04LOCK_LONGPADS -> SparkFun-Connectors:M04SCREW_LOCK
- JP20: value M01PTH -> (none); device SparkFun-Connectors:M01PTH -> SparkFun-Connectors:M04LOCK
- JP3: value I2C1-B -> SERVO; device SparkFun-Connectors:M04LOCK_LONGPADS -> SparkFun-Connectors:M03LOCK_LONGPADS
- JP4: value BATT -> ESCA; device SparkFun-Connectors:M023.5MM_LOCK -> SparkFun-Connectors:M03LOCK_LONGPADS
- JP5: value I2C1-A -> ESCB; device SparkFun-Connectors:M04LOCK_LONGPADS -> SparkFun-Connectors:M03LOCK_LONGPADS
- JP6: value UART2 -> ESCC; device SparkFun-Connectors:M04LOCK_LONGPADS -> SparkFun-Connectors:M03LOCK_LONGPADS
- JP7: value MOTORS -> ESCD; device SparkFun-Connectors:M04SCREW_LOCK -> SparkFun-Connectors:M03LOCK_LONGPADS
- JP8: value SPI1 -> USART1; device SparkFun-Connectors:M06LOCK_LONGPADS -> SparkFun-Connectors:M04LOCK_LONGPADS
- JP9: value SERVO -> I2C1-A; device SparkFun-Connectors:M03LOCK_LONGPADS -> SparkFun-Connectors:M04LOCK_LONGPADS
- LED2: value (none) -> GREEN
- LED3: value GREEN -> (none)
- R1: value 270 -> 10k
- R11: value 1k -> 270
- R12, R17, R18, R19: value 1k -> 50
- R13: value 1k -> 100
- R14: value 100 -> 1.5k
- R15: value 10k -> 1.5k
- R2, R6: value 1.5k -> 1k
- R3, R4, R5: value 50 -> 1k
- R7: value 50 -> 10k
- R8: value 10k -> 4.7k
- U2: value HMC5883LSMD -> VNH5019; device SparkFun-Sensors:HMC5883LSMD -> wicker:VNH5019
- U3: value STM32F4V -> MPU6000; device stm32f4:STM32F4V_100PIN_FOXCAR -> invensense:MPU-6000
- U4: value VNH5019 -> HMC5883LSMD; device wicker:VNH5019 -> SparkFun-Sensors:HMC5883LSMD
Connections:
- removed net N$13: C17.1, U6.REGOUT
- removed net N$17: JP34.1, U3.PC4
- removed net N$8: JP33.1, U3.PC5
- new net REGOUT: C8.1, U3.REGOUT
- net 3.3V: now also C13.1, C14.2, C15.2, C17.2, C22.2, C24.2, C4.1, C7.1, J1.VDD, J2.VCC, J2.VREF, JP10.4, JP11.4, JP12.4, JP13.6, JP3.2, JP8.4, JP9.4, LED2.A, R13.2, R15.2, R16.2, R17.1, R18.1, R19.1, U3.VDD, U4.S1, U4.VDD, U4.VDDIO, U5.VCAP_1, U5.VCAP_2, U5.VDD1, U5.VDD2, U5.VDD3, U5.VDD4, U5.VDD5, U5.VDD6, U5.VDDA; no longer C11.2, C14.1, C19.2, C22.1, C6.1, C7.2, C8.2, C9.2, J2.VDD, J3.VCC, J3.VREF, JP15.4, JP2.4, JP3.4, JP5.4, JP6.4, JP8.6, JP9.2, LED3.A, R2.2, R20.2, R3.1, R4.1, R5.1, R6.2, TP4.TP, U2.S1, U2.VDD, U2.VDDIO, U3.VCAP_1, U3.VCAP_2, U3.VDD1, U3.VDD2, U3.VDD3, U3.VDD4, U3.VDD5, U3.VDD6, U3.VDDA, U6.VDD
- net CP: now also U2.CP; no longer U4.CP
- net CS: now also R7.2, R9.2, U2.CS; no longer R11.2, R15.2, U4.CS
- net DIR: now also JP3.1, U5.PE11; no longer JP9.1, TP13.TP, U3.PE11
- net ENA: now also R10.1, R2.2, U2.ENA; no longer R18.2, R20.1, U4.ENA
- net ENB: now also R3.2, R8.1, U2.ENB; no longer R10.1, R13.2, U4.ENB
- net ESCA: now also JP4.1, U5.PE15; no longer JP14.1, TP11.TP, U3.PE15
- net ESCB: now also JP5.1, U5.PE14; no longer JP13.1, TP10.TP, U3.PE14
- net ESCC: now also JP6.1, U5.PE13; no longer JP12.1, TP9.TP, U3.PE13
- net ESCD: now also JP7.1, U5.PE12; no longer JP11.1, TP8.TP, U3.PE12
- net FS_DM: now also J3.D-, U5.PA11; no longer J1.D-, U3.PA11
- net FS_DP: now also J3.D+, U5.PA12; no longer J1.D+, U3.PA12
- net FS_ID: now also J3.ID, U5.PA10; no longer J1.ID, U3.PA10
- net FS_VBUS: now also J3.VCC, U5.PA9; no longer J1.VCC, U3.PA9
- net GND: now also C11.2, C14.1, C15.1, C16.1, C17.1, C22.1, C24.1, C4.2, C5.2, C7.2, C8.2, C9.2, J1.CARD_DETECT, J1.CARD_DETECT1, J1.GND1, J1.VSS, JP1.1, JP10.1, JP11.1, JP12.1, JP13.1, JP2.2, JP3.3, JP9.1, R12.1, R9.1, U2.GND, U3.CLKIN, U3.GND, U4.GND@1, U4.GND@2, U5.VREF+, U5.VSS1, U5.VSS2, U5.VSS3, U5.VSSA; no longer C11.1, C12.2, C14.2, C16.2, C17.2, C22.2, C24.2, C4.1, C5.1, C7.1, C8.1, C9.1, J2.CARD_DETECT, J2.CARD_DETECT1, J2.GND1, J2.VSS, JP15.1, JP2.1, JP3.1, JP4.1, JP5.1, JP6.1, JP7.2, JP9.3, R16.1, R7.1, U2.GND@1, U2.GND@2, U3.VREF+, U3.VSS1, U3.VSS2, U3.VSS3, U3.VSSA, U4.GND, U6.CLKIN, U6.GND
- net IMU_CLKOUT: now also U3.CLKOUT, U5.PD10; no longer U3.PD10, U6.CLKOUT
- net IMU_FSYNC: now also U3.FSYNC, U5.PD9; no longer U3.PD9, U6.FSYNC
- net IMU_INT: now also U3.INT, U5.PD8; no longer U3.PD8, U6.INT
- net INA: now also R4.2, U2.INA; no longer R19.2, U4.INA
- net INB: now also R5.2, U2.INB; no longer R12.2, U4.INB
- net LED_B: now also U5.PC15; no longer U3.PC15
- net LED_G: now also U5.PC14; no longer U3.PC14
- net LED_R: now also LED3.A, U5.PC13; no longer LED2.A, U3.PC13
- net MD_CS: now also C2.1, R7.1, U5.PB2; no longer C13.1, R15.1, U3.PB2
- net MD_CSDIS: now also U2.CS_DIS, U5.PE8; no longer U3.PE8, U4.CS_DIS
- net MD_ENA: now also R2.1, U5.PE9; no longer R18.1, U3.PE9
- net MD_ENB: now also R3.1, U5.PB1; no longer R13.1, U3.PB1
- net MD_INA: now also R4.1, U5.PE10; no longer R19.1, U3.PE10
- net MD_INB: now also R5.1, U5.PB0; no longer R12.1, U3.PB0
- net MD_PWM: now also R1.2, R6.1, U5.PE7; no longer R16.2, R17.1, U3.PE7
- net N$1: now also JP18.1, U5.PA8; no longer JP25.1, U3.PA8
- net N$10: now also JP17.3, U5.PC1; no longer JP37.1, U3.PC1
- net N$11: now also C12.1, U4.SETP; no longer C15.1, U2.SETP
- net N$12: now also C11.1, U4.C1; no longer C16.1, U2.C1
- net N$14: now also JP17.2, U5.PC2; no longer JP36.1, U3.PC2
- net N$15: now also JP19.1, U5.PE1; no longer JP1.1, U3.PE1
- net N$16: now also JP17.1, U5.PC3; no longer JP35.1, U3.PC3
- net N$18: now also C9.1, U3.CPOUT; no longer C24.1, U6.CPOUT
- net N$2: now also LED2.C, R12.2; no longer LED3.C, R7.2
- net N$20: now also R13.1; no longer R14.1
- net N$3: now also R11.2; no longer R1.2
- net N$4: now also C12.2, U4.SETC; no longer C15.2, U2.SETC
- net N$41: now also JP16.2, U5.PE2; no longer JP43.1, U3.PE2
- net N$42: now also JP16.1, U5.PE3; no longer JP42.1, U3.PE3
- net N$43: now also JP17.7, U5.PE4; no longer JP41.1, U3.PE4
- net N$44: now also JP17.6, U5.PE5; no longer JP40.1, U3.PE5
- net N$45: now also JP17.5, U5.PE6; no longer JP39.1, U3.PE6
- net N$5: now also LED3.C, R17.2; no longer LED2.C, R4.2
- net N$55: now also JP18.2, U5.PC7; no longer JP26.1, U3.PC7
- net N$56: now also JP18.3, U5.PC6; no longer JP27.1, U3.PC6
- net N$57: now also JP18.4, U5.PD15; no longer JP28.1, U3.PD15
- net N$58: now also JP18.5, U5.PD14; no longer JP29.1, U3.PD14
- net N$59: now also JP18.6, U5.PD13; no longer JP30.1, U3.PD13
- net N$6: now also R18.2; no longer R5.2
- net N$60: now also JP18.7, U5.PD12; no longer JP31.1, U3.PD12
- net N$61: now also JP18.8, U5.PD11; no longer JP32.1, U3.PD11
- net N$66: now also JP19.2, U5.PE0; no longer JP10.1, U3.PE0
- net N$67: now also JP14.1, U5.PB5; no longer JP16.1, U3.PB5
- net N$68: now also JP14.2, U5.PB4; no longer JP17.1, U3.PB4
- net N$69: now also JP14.3, U5.PD7; no longer JP18.1, U3.PD7
- net N$7: now also R19.2; no longer R3.2
- net N$70: now also JP14.4, U5.PD6; no longer JP19.1, U3.PD6
- net N$71: now also U5.PD5; no longer U3.PD5
- net N$72: now also JP20.2, U5.PD4; no longer JP21.1, U3.PD4
- net N$73: now also JP20.3, U5.PD3; no longer JP22.1, U3.PD3
- net N$74: now also JP20.4, U5.PD1; no longer JP23.1, U3.PD1
- net N$75: now also JP15.1, U5.PD0; no longer JP24.1, U3.PD0
- net N$9: now also JP17.4, U5.PC0; no longer JP38.1, U3.PC0
- net NRST: now also J2.!RESET, R16.1, U5.NRST; no longer J3.!RESET, R8.1, U3.NRST
- net OSC_IN1: now also C19.2, U5.PH0; no longer C4.2, U3.PH0
- net OSC_OUT1: now also C16.2, U5.PH1; no longer C5.2, U3.PH1
- net OUTA: now also JP2.4, U2.OUTA; no longer JP7.4, U4.OUTA
- net OUTB: now also JP2.3, U2.OUTB; no longer JP7.3, U4.OUTB
- net PWM: now also R6.2, U2.PWM; no longer R17.2, U4.PWM
- net RX1: now also JP8.2, U5.PA1; no longer JP2.2, U3.PA1
- net RX2: now also JP10.2, U5.PA3; no longer JP6.2, U3.PA3
- net RX3: now also JP12.2, U5.PB11; no longer JP15.2, U3.PB11
- net RX_DOUT1: now also J2.DOUT, U5.PB7; no longer J3.DOUT, U3.PB7
- net SCL1: now also JP11.2, JP9.2, R15.1, U4.SCL, U5.PB8; no longer JP3.2, JP5.2, R6.1, U2.SCL, U3.PB8
- net SDA1: now also JP11.3, JP9.3, R14.1, U4.SDA, U5.PB9; no longer JP3.3, JP5.3, R2.1, U2.SDA, U3.PB9
- net SDIO_CLK: now also J1.SCLK, U5.PC12; no longer J2.SCLK, U3.PC12
- net SDIO_CMD: now also J1.DATA_IN, U5.PD2; no longer J2.DATA_IN, U3.PD2
- net SDIO_D0: now also J1.DATA_OUT, U5.PC8; no longer J2.DATA_OUT, U3.PC8
- net SDIO_D1: now also J1.DAT1, U5.PC9; no longer J2.DAT1, U3.PC9
- net SDIO_D2: now also J1.DAT2, U5.PC10; no longer J2.DAT2, U3.PC10
- net SDIO_D3: now also J1.CS, U5.PC11; no longer J2.CS, U3.PC11
- net SPI1_MISO: now also JP13.3, U5.PA6; no longer JP8.3, U3.PA6
- net SPI1_MOSI: now also JP13.2, U5.PA7; no longer JP8.2, U3.PA7
- net SPI1_NSS: now also JP13.5, U5.PA4; no longer JP8.5, U3.PA4
- net SPI1_SCK: now also JP13.4, U5.PA5; no longer JP8.4, U3.PA5
- net SPI2_CS: now also U3.!CS, U5.PB12; no longer U3.PB12, U6.!CS
- net SPI2_MISO: now also U3.AD0/SDO, U5.PB14; no longer U3.PB14, U6.AD0/SDO
- net SPI2_MOSI: now also U3.SDA/SDI, U5.PB15; no longer U3.PB15, U6.SDA/SDI
- net SPI2_SCK: now also U3.SCL/SCLK, U5.PB13; no longer U3.PB13, U6.SCL/SCLK
- net TCK: now also U5.PA14; no longer U3.PA14
- net TDI: now also U5.PA15; no longer U3.PA15
- net TDO: now also U5.PB3; no longer U3.PB3
- net TMS: now also U5.PA13; no longer U3.PA13
- net TX1: now also JP8.3, U5.PA0; no longer JP2.3, U3.PA0
- net TX2: now also JP10.3, U5.PA2; no longer JP6.3, U3.PA2
- net TX3: now also JP12.3, U5.PB10; no longer JP15.3, U3.PB10
- net TX_DIN1: now also J2.DIN/!CONFIG, U5.PB6; no longer J3.DIN/!CONFIG, U3.PB6
- net VCC: now also C5.1, C6.1, U2.VCC; no longer C2.1, C3.1, U4.VCC
- net VIN: now also C3.1, JP1.2, JP2.1, U2.VBAT; no longer C12.1, JP4.2, JP7.1, TP3.TP, U4.VBAT
